File: AteGates/revisions/R1_0_0/AteGates.brd (EAGLE design)
At the start: 79.2 x 27.4 mm, 92 parts, among them J100 F10, J101 F10, P1J JACK-3_5MM-MONO-SW-WQP_PJ302-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, P2J JACK-3_5MM-MONO-SW-WQP_PJ302-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, P3J JACK-3_5MM-MONO-SW-WQP_PJ302-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, P4J JACK-3_5MM-MONO-SW-WQP_PJ302-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, P5J JACK-3_5MM-MONO-SW-WQP_PJ302-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, P6J JACK-3_5MM-MONO-SW-WQP_PJ302-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, P7J JACK-3_5MM-MONO-SW-WQP_PJ302-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, P8J JACK-3_5MM-MONO-SW-WQP_PJ302-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

Commit message: 4/10 update
Parts:
- removed R10: 47K, PatternAgents-ProtoPads:0603-RES
- removed R9: 33K, PatternAgents-ProtoPads:0603-RES
Connections:
- removed net 12V0: J101.6, R10.2
- removed net N12V0: J100.6
- net GND: no longer R9.1
- net VCC: now also J100.6, J101.6; no longer R10.1, R9.2
Routing:
- net GND: track 203.2 -> 188.4 mm, vias 5 -> 4
- net VCC: track 203.9 -> 211.8 mm
- net 12V0: track 2.52 -> 0.00 mm
Other:
- board text added: ""AteGates" Rev1.0"
- board text added: "PatternAgents.com "AteGates" Eight Gates I/O Board Rev 1.0"
- board text removed: ""AteGates" Rev3.0.0"
- board text removed: "PatternAgents.com "AteGates" Eight Gates I/O Board Rev 3.0.0"
